Commit message: Changed docker to access files as a bind rather than a copy, both faster and more reliable

File: ros2_ws/src/lunabot_2425/description/robot_core.xacro (robot description, xacro)
@@ -27,14 +27,14 @@
     <link name="chassis">
         <visual>
-            <origin xyz="0 0 0" rpy="0 0 0" />
-            <geometry>
-                <mesh filename="package://lunabot_2425/stl/chassis.stl" />
+            <origin xyz="0 0 0" rpy=" -1.57079632679489 -3.14159265358979 -1.57079632679489" />
+            <geometry>
+                <mesh filename="package://lunabot_2425/stl/bucket_meter.stl" />
             </geometry>
             <material name="white" />
         </visual>
         <collision>
-            <origin xyz="0 0 0" rpy="0 0 0" />
-            <geometry>
-                <mesh filename="package://lunabot_2425/stl/chassis.stl" />
+            <origin xyz="0 0 0" rpy=" -1.57079632679489 -3.14159265358979 -1.57079632679489" />
+            <geometry>
+                <mesh filename="package://lunabot_2425/stl/bucket_meter.stl" />
             </geometry>
         </collision>

Commit message: got xacro to work but is super overdetailed and runs slow. need to reduce part complexity aggresivley

File: ros2_ws/src/lunabot_2425/description/robot_core.xacro (robot description, xacro)
@@ -1,243 +1,339 @@
 <?xml version="1.0"?>
-<robot xmlns:xacro="http://www.ros.org/wiki/xacro">
-    <material name="white">
-        <color rgba="1 1 1 1" />
-    </material>
-    <material name="red">
-        <color rgba="0.8 0.1 0.1 1" />
-    </material>
-    <material name="grey">
-        <color rgba="0.7 0.7 0.7 1" />
-    </material>
-    <material name="green">
-        <color rgba="0.1 0.8 0.1 1" />
-    </material>
-    <material name="black">
-        <color rgba="0 0 0 1" />
-    </material>
-    <!-- BASE LINK -->
-    <link name="base_link">
-    </link>
-    <!-- CHASSIS LINK -->
-    <joint name="chassis_joint" type="fixed">
-        <parent link="base_link" />
-        <child link="chassis" />
-        <origin xyz="0 0 0.144" rpy="0 0 1.57079632679489" />
-    </joint>
-    <link name="chassis">
-        <visual>
-            <origin xyz="0 0 0" rpy=" -1.57079632679489 -3.14159265358979 -1.57079632679489" />
-            <geometry>
-                <mesh filename="package://lunabot_2425/stl/bucket_meter.stl" />
-            </geometry>
-            <material name="white" />
-        </visual>
-        <collision>
-            <origin xyz="0 0 0" rpy=" -1.57079632679489 -3.14159265358979 -1.57079632679489" />
-            <geometry>
-                <mesh filename="package://lunabot_2425/stl/bucket_meter.stl" />
-            </geometry>
-        </collision>
-        <inertial>
-            <origin xyz="0.00047255856824676841735 0.0223648596978729651 0.13076886029956547031" rpy="0 0 0"/>
-            <mass value="25" />
-            <inertia ixx="0.90389242187733576106" ixy="0.0034717089339218617193"  ixz="-0.0076346994671778805816" iyy="0.40577362837262359596" iyz="-0.068059613649222985843" izz="0.9121615213756760765" />
-        </inertial>
-    </link>
-    <!-- REAR LEFT WHEEL POD ASSEMBLY -->
-    <joint name="rear_left_steer_joint" type="continuous">
-        <parent link="chassis" />
-        <child link="rear_left_pod" />
-        <origin xyz="0.2655 0.2539125 0.0894" rpy="0 0 3.14159265358979" />
-        <axis xyz="0 0 1" />
-    </joint>
-    <link name="rear_left_pod">
-        <visual>
-            <geometry>
-                <mesh filename="package://lunabot_2425/stl/wheelpod.stl" />
-            </geometry>
-            <material name="red" />
-        </visual>
-        <collision>
-            <geometry>
-                <mesh filename="package://lunabot_2425/stl/wheelpod.stl" />
-            </geometry>
-        </collision>
-        <inertial>
-            <origin xyz="0.030048248825093670095 0 -0.054580062726334643841" rpy="0 0 0"/>
-            <mass value="0.5" />
-            <inertia ixx="0.0013087489021583560353" ixy="0"  ixz="0.00026671164402675704222" iyy="0.0013673630909145266868" iyz="0" izz="0.00042583920876048439019" />
-        </inertial>
-    </link>
-    <joint name="rear_left_drive_joint" type="continuous">
-        <parent link="rear_left_pod" />
-        <child link="rear_left_wheel" />
-        <origin xyz="0.0335 0 -0.13335" rpy="-1.57079632679489 0 3.14159265358979" />
-        <axis xyz="1 0 0"/>
-    </joint>
-    <link name="rear_left_wheel">
-        <visual>
-            <geometry>
-                <mesh filename="package://lunabot_2425/stl/wheel.stl" />
-            </geometry>
-            <material name="black" />
-        </visual>
-        <collision>
-            <geometry>
-                <mesh filename="package://lunabot_2425/stl/wheel.stl" />
-            </geometry>
-        </collision>
-        <inertial>
-            <origin xyz="0.03 0 0" rpy="0 0 0"/>
-            <mass value="1" />
-            <inertia ixx="0.0052" ixy="0" ixz="0" iyy="0.0029" iyz="0" izz="0.0029" />
-        </inertial>
-    </link>
-    <!-- REAR RIGHT WHEEL POD ASSEMBLY -->
-    <joint name="rear_right_steer_joint" type="continuous">
-        <parent link="chassis" />
-        <child link="rear_right_pod" />
-        <origin xyz="-0.2655 0.2539125 0.0894" rpy="0 0 0" />
-        <axis xyz="0 0 1" />
-    </joint>
-    <link name="rear_right_pod">
-        <visual>
-            <geometry>
-                <mesh filename="package://lunabot_2425/stl/wheelpod.stl" />
-            </geometry>
-            <material name="red" />
-        </visual>
-        <collision>
-            <geometry>
-                <mesh filename="package://lunabot_2425/stl/wheelpod.stl" />
-            </geometry>
-        </collision>
-        <inertial>
-            <origin xyz="0.030048248825093670095 0 -0.054580062726334643841" rpy="0 0 0"/>
-            <mass value="0.5" />
-            <inertia ixx="0.0013087489021583560353" ixy="0"  ixz="0.00026671164402675704222" iyy="0.0013673630909145266868" iyz="0" izz="0.00042583920876048439019" />
-        </inertial>
-    </link>
-    <joint name="rear_right_drive_joint" type="continuous">
-        <parent link="rear_right_pod" />
-        <child link="rear_right_wheel" />
-        <origin xyz="0.0335 0 -0.13335" rpy="-1.57079632679489 0 3.14159265358979" />
-        <axis xyz="-1 0 0"/>
-    </joint>
-    <link name="rear_right_wheel">
-        <visual>
-            <geometry>
-                <mesh filename="package://lunabot_2425/stl/wheel.stl" />
-            </geometry>
-            <material name="black" />
-        </visual>
-        <collision>
-            <geometry>
-                <mesh filename="package://lunabot_2425/stl/wheel.stl" />
-            </geometry>
-        </collision>
-        <inertial>
-            <origin xyz="0.03 0 0" rpy="0 0 0"/>
-            <mass value="1" />
-            <inertia ixx="0.0052" ixy="0" ixz="0" iyy="0.0029" iyz="0" izz="0.0029" />
-        </inertial>
-    </link>
-    <!-- FRONT LEFT WHEEL POD ASSEMBLY -->
-    <joint name="front_left_steer_joint" type="continuous">
-        <parent link="chassis" />
-        <child link="front_left_pod" />
-        <origin xyz="0.2655 -0.2539125 0.0894" rpy="0 0 3.14159265358979" />
-        <axis xyz="0 0 1" />
-    </joint>
-    <link name="front_left_pod">
-        <visual>
-            <geometry>
-                <mesh filename="package://lunabot_2425/stl/wheelpod.stl" />
-            </geometry>
-            <material name="red" />
-        </visual>
-        <collision>
-            <geometry>
-                <mesh filename="package://lunabot_2425/stl/wheelpod.stl" />
-            </geometry>
-        </collision>
-        <inertial>
-            <origin xyz="0.030048248825093670095 0 -0.054580062726334643841" rpy="0 0 0"/>
-            <mass value="0.5" />
-            <inertia ixx="0.0013087489021583560353" ixy="0"  ixz="0.00026671164402675704222" iyy="0.0013673630909145266868" iyz="0" izz="0.00042583920876048439019" />
-        </inertial>
-    </link>
-    <joint name="front_left_drive_joint" type="continuous">
-        <parent link="front_left_pod" />
-        <child link="front_left_wheel" />
-        <origin xyz="0.0335 0 -0.13335" rpy="-1.57079632679489 0 3.14159265358979" />
-        <axis xyz="1 0 0"/>
-    </joint>
-    <link name="front_left_wheel">
-        <visual>
-            <geometry>
-                <mesh filename="package://lunabot_2425/stl/wheel.stl" />
-            </geometry>
-            <material name="black" />
-        </visual>
-        <collision>
-            <geometry>
-                <mesh filename="package://lunabot_2425/stl/wheel.stl" />
-            </geometry>
-        </collision>
-        <inertial>
-            <origin xyz="0.03 0 0" rpy="0 0 0"/>
-            <mass value="1" />
-            <inertia ixx="0.0052" ixy="0" ixz="0" iyy="0.0029" iyz="0" izz="0.0029" />
-        </inertial>
-    </link>
-    <!-- FRONT RIGHT WHEEL POD ASSEMBLY -->
-    <joint name="front_right_steer_joint" type="continuous">
-        <parent link="chassis" />
-        <child link="front_right_pod" />
-        <origin xyz="-0.2655 -0.2539125 0.0894" rpy="0 0 0" />
-        <axis xyz="0 0 1" />
-    </joint>
-    <link name="front_right_pod">
-        <visual>
-            <geometry>
-                <mesh filename="package://lunabot_2425/stl/wheelpod.stl" />
-            </geometry>
-            <material name="red" />
-        </visual>
-        <collision>
-            <geometry>
-                <mesh filename="package://lunabot_2425/stl/wheelpod.stl" />
-            </geometry>
-        </collision>
-        <inertial>
-            <origin xyz="0.030048248825093670095 0 -0.054580062726334643841" rpy="0 0 0"/>
-            <mass value="0.5" />
-            <inertia ixx="0.0013087489021583560353" ixy="0"  ixz="0.00026671164402675704222" iyy="0.0013673630909145266868" iyz="0" izz="0.00042583920876048439019" />
-        </inertial>
-    </link>
-    <joint name="front_right_drive_joint" type="continuous">
-        <parent link="front_right_pod" />
-        <child link="front_right_wheel" />
-        <origin xyz="0.0335 0 -0.13335" rpy="-1.57079632679489 0 3.14159265358979" />
-        <axis xyz="-1 0 0"/>
-    </joint>
-    <link name="front_right_wheel">
-        <visual>
-            <geometry>
-                <mesh filename="package://lunabot_2425/stl/wheel.stl" />
-            </geometry>
-            <material name="black" />
-        </visual>
-        <collision>
-            <geometry>
-                <mesh filename="package://lunabot_2425/stl/wheel.stl" />
-            </geometry>
-        </collision>
-        <inertial>
-            <origin xyz="0.03 0 0" rpy="0 0 0"/>
-            <mass value="1" />
-            <inertia ixx="0.0052" ixy="0" ixz="0" iyy="0.0029" iyz="0" izz="0.0029" />
-        </inertial>
-    </link>
+<robot name="lunabot" xmlns:xacro="http://www.ros.org/wiki/xacro">
+  <xacro:property name="deg180" value="3.14159265"/>
+  <xacro:property name="deg90" value="1.5707963"/>
+  <xacro:property name="brx" value="0"/>
+  <xacro:property name="bry" value="0.126975"/>
+  <xacro:property name="brz" value="0.229093"/>
+  <xacro:property name="rkx" value="0.254"/>
+  <xacro:property name="rky" value="0.019"/>
+  <xacro:property name="rkz" value="0.139725"/>
+  <xacro:property name="kwx" value="0"/>
+  <xacro:property name="kwy" value="-0.038135"/>
+  <xacro:property name="kwz" value="-0.146383"/>
+  <!-- MATERIALS -->
+  <material name="grey">
+    <color rgba="0.7 0.7 0.7 1"/>
+  </material>
+  <material name="green">
+    <color rgba="0.6 0.2 0.5 1"/>
+  </material>
+  <material name="blue">
+    <color rgba="0.1 0.1 0.7 1"/>
+  </material>
+  <material name="red">
+    <color rgba="0.7 0.1 0.1 1"/>
+  </material>
+  <material name="gold">
+    <color rgba="0.83 0.67 0.2 1"/>
+  </material>
+  <!-- BASE LINK -->
+  <link name="base_link">
+    <inertial>
+      <mass value="1.0"/>
+      <origin xyz="0 0 0" rpy="0 0 0"/>
+      <inertia ixx="0.01" ixy="0" ixz="0" iyy="0.01" iyz="0" izz="0.01"/>
+    </inertial>
+  </link>
+  <!-- BUCKET -->
+  <link name="bucket">
+    <visual>
+      <geometry>
+        <mesh filename="package://lunabot_2425/stl/bucket_mo.stl"/>
+      </geometry>
+      <origin xyz="0 0 0" rpy="0 0 0"/>
+      <material name="green"/>
+    </visual>
+    <collision>
+      <geometry>
+        <mesh filename="package://lunabot_2425/stl/bucket_mo.stl"/>
+      </geometry>
+      <origin xyz="0 0 0" rpy="0 0 0"/>
+    </collision>
+    <inertial>
+      <mass value="15"/>
+      <origin xyz="0 0 0" rpy="0 0 0"/>
+      <inertia ixx="0.9" ixy="0" ixz="0" iyy="0.4" iyz="0" izz="0.9"/>
+    </inertial>
+  </link>
+  <!-- BUCKET JOINT -->
+  <joint name="bucket_joint" type="fixed">
+    <parent link="base_link"/>
+    <child link="bucket"/>
+    <origin xyz="0 0 0" rpy="0 0 0"/>
+  </joint>
+  <!-- LEFT ROCKER -->
+  <link name="left_rocker">
+    <visual>
+      <geometry>
+        <mesh filename="package://lunabot_2425/stl/left_rocker_mo.stl"/>
+      </geometry>
+      <origin xyz="0 0 0" rpy="0 0 0"/>
+      <material name="blue"/>
+    </visual>
+    <collision>
+      <geometry>
+        <mesh filename="package://lunabot_2425/stl/left_rocker_mo.stl"/>
+      </geometry>
+      <origin xyz="0 0 0" rpy="0 0 0"/>
+    </collision>
+    <inertial>
+      <mass value="5"/>
+      <origin xyz="0 0 0" rpy="0 0 0"/>
+      <inertia ixx="0.01" ixy="0" ixz="0" iyy="0.01" iyz="0" izz="0.01"/>
+    </inertial>
+  </link>
+  <!-- LEFT ROCKER JOINT -->
+  <joint name="left_rocker_joint" type="fixed">
+    <parent link="bucket"/>
+    <child link="left_rocker"/>
+    <origin xyz="${brx} ${bry} ${brz}" rpy="-${deg90} ${deg180} 0"/>
+  </joint>
+  <!-- RIGHT ROCKER -->
+  <link name="right_rocker">
+    <visual>
+      <geometry>
+        <mesh filename="package://lunabot_2425/stl/right_rocker_mo.stl"/>
+      </geometry>
+      <origin xyz="0 0 0" rpy="0 0 0"/>
+      <material name="blue"/>
+    </visual>
+    <collision>
+      <geometry>
+        <mesh filename="package://lunabot_2425/stl/right_rocker_mo.stl"/>
+      </geometry>
+      <origin xyz="0 0 0" rpy="0 0 0"/>
+    </collision>
+    <inertial>
+      <mass value="5"/>
+      <origin xyz="0 0 0" rpy="0 0 0"/>
+      <inertia ixx="0.01" ixy="0" ixz="0" iyy="0.01" iyz="0" izz="0.01"/>
+    </inertial>
+  </link>
+  <!-- RIGHT ROCKER JOINT -->
+  <joint name="right_rocker_joint" type="fixed">
+    <parent link="bucket"/>
+    <child link="right_rocker"/>
+    <origin xyz="${brx} -${bry} ${brz}" rpy="${deg90} 0 0"/>
+  </joint>
+  <!-- FRONT LEFT WHEEL POD -->
+  <!-- FRONT LEFT KNUCKLE -->
+  <link name="front_left_knuckle">
+    <visual>
+      <geometry>
+        <mesh filename="package://lunabot_2425/stl/knuckle_mo.stl"/>
+      </geometry>
+      <origin xyz="0 0 0" rpy="0 0 0"/>
+      <material name="gold"/>
+    </visual>
+    <collision>
+      <geometry>
+        <mesh filename="package://lunabot_2425/stl/knuckle_mo.stl"/>
+      </geometry>
+      <origin xyz="0 0 0" rpy="0 0 0"/>
+    </collision>
+    <inertial>
+      <mass value="2.0"/>
+      <origin xyz="0 0 0" rpy="0 0 0"/>
+      <inertia ixx="0.01" ixy="0" ixz="0" iyy="0.01" iyz="0" izz="0.01"/>
+    </inertial>
+  </link>
+  <!-- FRONT LEFT STEER JOINT -->
+  <joint name="front_left_steer_joint" type="fixed">
+    <parent link="left_rocker"/>
+    <child link="front_left_knuckle"/>
+    <origin xyz="-${rkx} ${rky} ${rkz}" rpy="-${deg90} ${deg180} 0"/>
+  </joint>
+  <!-- FRONT LEFT WHEEL -->
+  <link name="front_left_wheel">
+    <visual>
+      <geometry>
+        <mesh filename="package://lunabot_2425/stl/wheel_mo.stl"/>
+      </geometry>
+      <origin xyz="0 0 0" rpy="0 0 0"/>
+      <material name="red"/>
+    </visual>
+    <collision>
+      <geometry>
+        <mesh filename="package://lunabot_2425/stl/wheel_mo.stl"/>
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