Commit message: robot_core.xacro is dimensioned with properties

File: ros2_ws/src/lunabot_2425/description/robot_core.xacro (robot description, xacro)
@@ -3,13 +3,45 @@
   <xacro:property name="deg180" value="3.14159265"/>
   <xacro:property name="deg90" value="1.5707963"/>
+  <!-- BASE ROCKER Transform -->
   <xacro:property name="brx" value="0"/>
   <xacro:property name="bry" value="0.126975"/>
   <xacro:property name="brz" value="0.229093"/>
+  <!-- ROCKER KNUCKLE Transform -->
   <xacro:property name="rkx" value="0.254"/>
   <xacro:property name="rky" value="0.019"/>
   <xacro:property name="rkz" value="0.139725"/>
+  <!-- KNUCKLE WHEEL Transform -->
   <xacro:property name="kwx" value="0"/>
   <xacro:property name="kwy" value="-0.038135"/>
   <xacro:property name="kwz" value="-0.146383"/>
+  <!-- BUCKET Dimensions -->
+  <xacro:property name="buck_sx" value="0.65"/>
+  <xacro:property name="buck_sy" value="0.25"/>
+  <xacro:property name="buck_sz" value="0.30"/>
+  <xacro:property name="buck_px" value="-0.1"/>
+  <xacro:property name="buck_py" value="0"/>
+  <xacro:property name="buck_pz" value="0.295"/>
+  <!-- Rocker Dimensions -->
+  <xacro:property name="rock_rad" value="0.025"/>
+  <xacro:property name="rock_len" value="0.55"/>
+  <xacro:property name="rock_px" value="0"/>
+  <xacro:property name="rock_py" value="0.05"/>
+  <xacro:property name="rock_pz" value="0.075"/>
+  <xacro:property name="rock_rx" value="0"/>
+  <xacro:property name="rock_ry" value="${deg90}"/>
+  <xacro:property name="rock_rz" value="0"/>
+  <!-- KNUCKLE Dimensions -->
+  <xacro:property name="nuck_sx" value="0.0675"/>
+  <xacro:property name="nuck_sy" value="0.035"/>
+  <xacro:property name="nuck_sz" value="0.15"/>
+  <xacro:property name="nuck_px" value="0"/>
+  <xacro:property name="nuck_py" value="-0.065"/>
+  <xacro:property name="nuck_pz" value="-0.075"/>
+  <!-- WHEEL Dimensions -->
+  <xacro:property name="whee_rad" value="0.1"/>
+  <xacro:property name="whee_len" value="0.075"/>
+  <xacro:property name="whee_px" value="0"/>
+  <xacro:property name="whee_py" value="0"/>
+  <xacro:property name="whee_pz" value="0.035"/>
   <!-- MATERIALS -->
   <material name="grey">
@@ -40,14 +72,16 @@
     <visual>
       <geometry>
-        <mesh filename="package://lunabot_2425/stl/bucket_mo.stl"/>
-      </geometry>
-      <origin xyz="0 0 0" rpy="0 0 0"/>
+        <!-- <mesh filename="package://lunabot_2425/stl/bucket_mo.stl"/> -->
+        <box size="${buck_sx} ${buck_sy} ${buck_sz}"/>
+      </geometry>
+      <origin xyz="${buck_px} ${buck_py} ${buck_pz}" rpy="0 0 0"/>
       <material name="green"/>
     </visual>
     <collision>
       <geometry>
-        <mesh filename="package://lunabot_2425/stl/bucket_mo.stl"/>
-      </geometry>
-      <origin xyz="0 0 0" rpy="0 0 0"/>
+        <!-- <mesh filename="package://lunabot_2425/stl/bucket_mo.stl"/> -->
+        <box size="${buck_sx} ${buck_sy} ${buck_sz}"/>
+      </geometry>
+      <origin xyz="${buck_px} ${buck_py} ${buck_pz}" rpy="0 0 0"/>
     </collision>
     <inertial>
@@ -67,18 +101,20 @@
     <visual>
       <geometry>
-        <mesh filename="package://lunabot_2425/stl/left_rocker_mo.stl"/>
-      </geometry>
-      <origin xyz="0 0 0" rpy="0 0 0"/>
+        <!-- <mesh filename="package://lunabot_2425/stl/left_rocker_mo.stl"/> -->
+        <cylinder radius="${rock_rad}" length="${rock_len}"/>
+      </geometry>
+      <origin xyz="${rock_px} ${rock_py} ${rock_pz}" rpy="${rock_rx} ${rock_ry} ${rock_rz}"/>
       <material name="blue"/>
     </visual>
     <collision>
       <geometry>
-        <mesh filename="package://lunabot_2425/stl/left_rocker_mo.stl"/>
-      </geometry>
-      <origin xyz="0 0 0" rpy="0 0 0"/>
+        <!-- <mesh filename="package://lunabot_2425/stl/left_rocker_mo.stl"/> -->
+        <cylinder radius="${rock_rad}" length="${rock_len}"/>
+      </geometry>
+      <origin xyz="${rock_px} ${rock_py} ${rock_pz}" rpy="${rock_rx} ${rock_ry} ${rock_rz}"/>
     </collision>
     <inertial>
       <mass value="5"/>
-      <origin xyz="0 0 0" rpy="0 0 0"/>
+      <origin xyz="${rock_px} ${rock_py} ${rock_pz}" rpy="${rock_rx} ${rock_ry} ${rock_rz}"/>
       <inertia ixx="0.01" ixy="0" ixz="0" iyy="0.01" iyz="0" izz="0.01"/>
     </inertial>
@@ -94,18 +130,20 @@
     <visual>
       <geometry>
-        <mesh filename="package://lunabot_2425/stl/right_rocker_mo.stl"/>
-      </geometry>
-      <origin xyz="0 0 0" rpy="0 0 0"/>
+        <!-- <mesh filename="package://lunabot_2425/stl/right_rocker_mo.stl"/> -->
+        <cylinder radius="${rock_rad}" length="${rock_len}"/>
+      </geometry>
+      <origin xyz="${rock_px} ${rock_py} ${rock_pz}" rpy="${rock_rx} ${rock_ry} ${rock_rz}"/>
       <material name="blue"/>
     </visual>
     <collision>
       <geometry>
-        <mesh filename="package://lunabot_2425/stl/right_rocker_mo.stl"/>
-      </geometry>
-      <origin xyz="0 0 0" rpy="0 0 0"/>
+        <!-- <mesh filename="package://lunabot_2425/stl/right_rocker_mo.stl"/> -->
+        <cylinder radius="${rock_rad}" length="${rock_len}"/>
+      </geometry>
+      <origin xyz="${rock_px} ${rock_py} ${rock_pz}" rpy="${rock_rx} ${rock_ry} ${rock_rz}"/>
     </collision>
     <inertial>
       <mass value="5"/>
-      <origin xyz="0 0 0" rpy="0 0 0"/>
+      <origin xyz="${rock_px} ${rock_py} ${rock_pz}" rpy="${rock_rx} ${rock_ry} ${rock_rz}"/>
       <inertia ixx="0.01" ixy="0" ixz="0" iyy="0.01" iyz="0" izz="0.01"/>
     </inertial>
@@ -122,18 +160,20 @@
     <visual>
       <geometry>
-        <mesh filename="package://lunabot_2425/stl/knuckle_mo.stl"/>
-      </geometry>
-      <origin xyz="0 0 0" rpy="0 0 0"/>
+        <!-- <mesh filename="package://lunabot_2425/stl/knuckle_mo.stl"/> -->
+        <box size="${nuck_sx} ${nuck_sy} ${nuck_sz}"/>
+      </geometry>
+      <origin xyz="${nuck_px} ${nuck_py} ${nuck_pz}" rpy="0 0 0"/>
       <material name="gold"/>
     </visual>
     <collision>
       <geometry>
-        <mesh filename="package://lunabot_2425/stl/knuckle_mo.stl"/>
-      </geometry>
-      <origin xyz="0 0 0" rpy="0 0 0"/>
-    </collision>
-    <inertial>
-      <mass value="2.0"/>
-      <origin xyz="0 0 0" rpy="0 0 0"/>
+        <!-- <mesh filename="package://lunabot_2425/stl/knuckle_mo.stl"/> -->
+        <box size="${nuck_sx} ${nuck_sy} ${nuck_sz}"/>
+      </geometry>
+      <origin xyz="${nuck_px} ${nuck_py} ${nuck_pz}" rpy="0 0 0"/>
+    </collision>
+    <inertial>
+      <mass value="2.0"/>
+      <origin xyz="${nuck_px} ${nuck_py} ${nuck_pz}" rpy="0 0 0"/>
       <inertia ixx="0.01" ixy="0" ixz="0" iyy="0.01" iyz="0" izz="0.01"/>
     </inertial>
@@ -149,18 +189,20 @@
     <visual>
       <geometry>
-        <mesh filename="package://lunabot_2425/stl/wheel_mo.stl"/>
-      </geometry>
-      <origin xyz="0 0 0" rpy="0 0 0"/>
+        <!-- <mesh filename="package://lunabot_2425/stl/wheel_mo.stl"/> -->
+        <cylinder radius="${whee_rad}" length="${whee_len}"/>
+      </geometry>
+      <origin xyz="${whee_px} ${whee_py} ${whee_pz}" rpy="0 0 0"/>
       <material name="red"/>
     </visual>
     <collision>
       <geometry>
-        <mesh filename="package://lunabot_2425/stl/wheel_mo.stl"/>
-      </geometry>
-      <origin xyz="0 0 0" rpy="0 0 0"/>
-    </collision>
-    <inertial>
-      <mass value="2.0"/>
-      <origin xyz="0 0 0" rpy="0 0 0"/>
+        <!-- <mesh filename="package://lunabot_2425/stl/wheel_mo.stl"/> -->
+        <cylinder radius="${whee_rad}" length="${whee_len}"/>
+      </geometry>
+      <origin xyz="${whee_px} ${whee_py} ${whee_pz}" rpy="0 0 0"/>
+    </collision>
+    <inertial>
+      <mass value="2.0"/>
+      <origin xyz="${whee_px} ${whee_py} ${whee_pz}" rpy="0 0 0"/>
       <inertia ixx="0.01" ixy="0" ixz="0" iyy="0.01" iyz="0" izz="0.01"/>
     </inertial>
@@ -177,18 +219,20 @@
     <visual>
       <geometry>
-        <mesh filename="package://lunabot_2425/stl/knuckle_mo.stl"/>
-      </geometry>
-      <origin xyz="0 0 0" rpy="0 0 0"/>
+        <!-- <mesh filename="package://lunabot_2425/stl/knuckle_mo.stl"/> -->
+        <box size="${nuck_sx} ${nuck_sy} ${nuck_sz}"/>
+      </geometry>
+      <origin xyz="${nuck_px} ${nuck_py} ${nuck_pz}" rpy="0 0 0"/>
       <material name="gold"/>
     </visual>
     <collision>
       <geometry>
-        <mesh filename="package://lunabot_2425/stl/knuckle_mo.stl"/>
-      </geometry>
-      <origin xyz="0 0 0" rpy="0 0 0"/>
-    </collision>
-    <inertial>
-      <mass value="2.0"/>
-      <origin xyz="0 0 0" rpy="0 0 0"/>
+        <!-- <mesh filename="package://lunabot_2425/stl/knuckle_mo.stl"/> -->
+        <box size="${nuck_sx} ${nuck_sy} ${nuck_sz}"/>
+      </geometry>
+      <origin xyz="${nuck_px} ${nuck_py} ${nuck_pz}" rpy="0 0 0"/>
+    </collision>
+    <inertial>
+      <mass value="2.0"/>
+      <origin xyz="${nuck_px} ${nuck_py} ${nuck_pz}" rpy="0 0 0"/>
       <inertia ixx="0.01" ixy="0" ixz="0" iyy="0.01" iyz="0" izz="0.01"/>
     </inertial>
@@ -204,18 +248,20 @@
     <visual>
       <geometry>
-        <mesh filename="package://lunabot_2425/stl/wheel_mo.stl"/>
-      </geometry>
-      <origin xyz="0 0 0" rpy="0 0 0"/>
+        <!-- <mesh filename="package://lunabot_2425/stl/wheel_mo.stl"/> -->
+        <cylinder radius="${whee_rad}" length="${whee_len}"/>
+      </geometry>
+      <origin xyz="${whee_px} ${whee_py} ${whee_pz}" rpy="0 0 0"/>
       <material name="red"/>
     </visual>
     <collision>
       <geometry>
-        <mesh filename="package://lunabot_2425/stl/wheel_mo.stl"/>
-      </geometry>
-      <origin xyz="0 0 0" rpy="0 0 0"/>
-    </collision>
-    <inertial>
-      <mass value="2.0"/>
-      <origin xyz="0 0 0" rpy="0 0 0"/>
+        <!-- <mesh filename="package://lunabot_2425/stl/wheel_mo.stl"/> -->
+        <cylinder radius="${whee_rad}" length="${whee_len}"/>
+      </geometry>
+      <origin xyz="${whee_px} ${whee_py} ${whee_pz}" rpy="0 0 0"/>
+    </collision>
+    <inertial>
+      <mass value="2.0"/>
+      <origin xyz="${whee_px} ${whee_py} ${whee_pz}" rpy="0 0 0"/>
       <inertia ixx="0.01" ixy="0" ixz="0" iyy="0.01" iyz="0" izz="0.01"/>
     </inertial>
@@ -232,18 +278,20 @@
     <visual>
       <geometry>
-        <mesh filename="package://lunabot_2425/stl/knuckle_mo.stl"/>
-      </geometry>
-      <origin xyz="0 0 0" rpy="0 0 0"/>
+        <!-- <mesh filename="package://lunabot_2425/stl/knuckle_mo.stl"/> -->
+        <box size="${nuck_sx} ${nuck_sy} ${nuck_sz}"/>
+      </geometry>
+      <origin xyz="${nuck_px} ${nuck_py} ${nuck_pz}" rpy="0 0 0"/>
       <material name="gold"/>
     </visual>
     <collision>
       <geometry>
-        <mesh filename="package://lunabot_2425/stl/knuckle_mo.stl"/>
-      </geometry>
-      <origin xyz="0 0 0" rpy="0 0 0"/>
-    </collision>
-    <inertial>
-      <mass value="2.0"/>
-      <origin xyz="0 0 0" rpy="0 0 0"/>
+        <!-- <mesh filename="package://lunabot_2425/stl/knuckle_mo.stl"/> -->
+        <box size="${nuck_sx} ${nuck_sy} ${nuck_sz}"/>
+      </geometry>
+      <origin xyz="${nuck_px} ${nuck_py} ${nuck_pz}" rpy="0 0 0"/>
+    </collision>
+    <inertial>
+      <mass value="2.0"/>
+      <origin xyz="${nuck_px} ${nuck_py} ${nuck_pz}" rpy="0 0 0"/>
       <inertia ixx="0.01" ixy="0" ixz="0" iyy="0.01" iyz="0" izz="0.01"/>
     </inertial>
@@ -259,18 +307,20 @@
     <visual>
       <geometry>
-        <mesh filename="package://lunabot_2425/stl/wheel_mo.stl"/>
-      </geometry>
-      <origin xyz="0 0 0" rpy="0 0 0"/>
+        <!-- <mesh filename="package://lunabot_2425/stl/wheel_mo.stl"/> -->
+        <cylinder radius="${whee_rad}" length="${whee_len}"/>
+      </geometry>
+      <origin xyz="${whee_px} ${whee_py} ${whee_pz}" rpy="0 0 0"/>
       <material name="red"/>
     </visual>
     <collision>
       <geometry>
-        <mesh filename="package://lunabot_2425/stl/wheel_mo.stl"/>
-      </geometry>
-      <origin xyz="0 0 0" rpy="0 0 0"/>
-    </collision>
-    <inertial>
-      <mass value="2.0"/>
-      <origin xyz="0 0 0" rpy="0 0 0"/>
+        <!-- <mesh filename="package://lunabot_2425/stl/wheel_mo.stl"/> -->
+        <cylinder radius="${whee_rad}" length="${whee_len}"/>
+      </geometry>
+      <origin xyz="${whee_px} ${whee_py} ${whee_pz}" rpy="0 0 0"/>
+    </collision>
+    <inertial>
+      <mass value="2.0"/>
+      <origin xyz="${whee_px} ${whee_py} ${whee_pz}" rpy="0 0 0"/>
       <inertia ixx="0.01" ixy="0" ixz="0" iyy="0.01" iyz="0" izz="0.01"/>
     </inertial>
@@ -287,18 +337,20 @@
     <visual>
       <geometry>
-        <mesh filename="package://lunabot_2425/stl/knuckle_mo.stl"/>
-      </geometry>
-      <origin xyz="0 0 0" rpy="0 0 0"/>
+        <!-- <mesh filename="package://lunabot_2425/stl/knuckle_mo.stl"/> -->
+        <box size="${nuck_sx} ${nuck_sy} ${nuck_sz}"/>
+      </geometry>
+      <origin xyz="${nuck_px} ${nuck_py} ${nuck_pz}" rpy="0 0 0"/>
       <material name="gold"/>
     </visual>
     <collision>
       <geometry>
-        <mesh filename="package://lunabot_2425/stl/knuckle_mo.stl"/>
-      </geometry>
-      <origin xyz="0 0 0" rpy="0 0 0"/>
-    </collision>
-    <inertial>
-      <mass value="2.0"/>
-      <origin xyz="0 0 0" rpy="0 0 0"/>
+        <!-- <mesh filename="package://lunabot_2425/stl/knuckle_mo.stl"/> -->
+        <box size="${nuck_sx} ${nuck_sy} ${nuck_sz}"/>
+      </geometry>
+      <origin xyz="${nuck_px} ${nuck_py} ${nuck_pz}" rpy="0 0 0"/>
+    </collision>
+    <inertial>
+      <mass value="2.0"/>
+      <origin xyz="${nuck_px} ${nuck_py} ${nuck_pz}" rpy="0 0 0"/>
       <inertia ixx="0.01" ixy="0" ixz="0" iyy="0.01" iyz="0" izz="0.01"/>
     </inertial>
@@ -314,18 +366,20 @@
     <visual>
       <geometry>
-        <mesh filename="package://lunabot_2425/stl/wheel_mo.stl"/>
-      </geometry>
-      <origin xyz="0 0 0" rpy="0 0 0"/>
+        <!-- <mesh filename="package://lunabot_2425/stl/wheel_mo.stl"/> -->
+        <cylinder radius="${whee_rad}" length="${whee_len}"/>
+      </geometry>
+      <origin xyz="${whee_px} ${whee_py} ${whee_pz}" rpy="0 0 0"/>
       <material name="red"/>
     </visual>
     <collision>
       <geometry>
-        <mesh filename="package://lunabot_2425/stl/wheel_mo.stl"/>
-      </geometry>
-      <origin xyz="0 0 0" rpy="0 0 0"/>
-    </collision>
-    <inertial>
-      <mass value="2.0"/>
-      <origin xyz="0 0 0" rpy="0 0 0"/>
+        <!-- <mesh filename="package://lunabot_2425/stl/wheel_mo.stl"/> -->
+        <cylinder radius="${whee_rad}" length="${whee_len}"/>
+      </geometry>
+      <origin xyz="${whee_px} ${whee_py} ${whee_pz}" rpy="0 0 0"/>
+    </collision>
+    <inertial>
+      <mass value="2.0"/>
+      <origin xyz="${whee_px} ${whee_py} ${whee_pz}" rpy="0 0 0"/>
       <inertia ixx="0.01" ixy="0" ixz="0" iyy="0.01" iyz="0" izz="0.01"/>
     </inertial>

Commit message: robot can be driven in simulation, axes are funky so turning is broken, gonna attempt to make an all new controller for quadruplex swerve

File: ros2_ws/src/lunabot_2425/description/robot_core.xacro (robot description, xacro)
@@ -180,8 +180,9 @@
   </link>
   <!-- FRONT LEFT STEER JOINT -->
-  <joint name="front_left_steer_joint" type="fixed">
+  <joint name="front_left_steer_joint" type="continuous">
     <parent link="left_rocker"/>
     <child link="front_left_knuckle"/>
     <origin xyz="-${rkx} ${rky} ${rkz}" rpy="-${deg90} ${deg180} 0"/>
+    <axis xyz="0 0 1"/>
   </joint>
   <!-- FRONT LEFT WHEEL -->
@@ -209,8 +210,9 @@
   </link>
   <!-- FRONT LEFT DRIVE JOINT -->
-  <joint name="front_left_drive_joint" type="fixed">
+  <joint name="front_left_drive_joint" type="continuous">
     <parent link="front_left_knuckle"/>
     <child link="front_left_wheel"/>
     <origin xyz="${kwx} ${kwy} ${kwz}" rpy="${deg90} 0 ${deg180}"/>
+    <axis xyz="0 0 1"/>
   </joint>
   <!-- FRONT RIGHT WHEEL POD -->
@@ -239,8 +241,9 @@
   </link>
   <!-- FRONT RIGHT STEER JOINT -->
-  <joint name="front_right_steer_joint" type="fixed">
+  <joint name="front_right_steer_joint" type="continuous">
     <parent link="right_rocker"/>
     <child link="front_right_knuckle"/>
     <origin xyz="${rkx} ${rky} ${rkz}" rpy="${deg90} 0 ${deg180}"/>
+    <axis xyz="0 0 1"/>
   </joint>
   <!-- FRONT RIGHT WHEEL -->
@@ -268,8 +271,9 @@
   </link>
   <!-- FRONT RIGHT DRIVE JOINT -->
-  <joint name="front_right_drive_joint" type="fixed">
+  <joint name="front_right_drive_joint" type="continuous">
     <parent link="front_right_knuckle"/>
     <child link="front_right_wheel"/>
     <origin xyz="${kwx} ${kwy} ${kwz}" rpy="${deg90} 0 ${deg180}"/>
+    <axis xyz="0 0 -1"/>
   </joint>
   <!-- BACK LEFT WHEEL POD -->
@@ -298,8 +302,9 @@
   </link>
   <!-- BACK LEFT STEER JOINT -->
-  <joint name="back_left_steer_joint" type="fixed">
+  <joint name="back_left_steer_joint" type="continuous">
     <parent link="left_rocker"/>
     <child link="back_left_knuckle"/>
     <origin xyz="${rkx} ${rky} ${rkz}" rpy="${deg90} 0 ${deg180}"/>
+    <axis xyz="0 0 1"/>
   </joint>
     <!-- BACK LEFT WHEEL -->
@@ -327,8 +332,9 @@
   </link>
   <!-- BACK LEFT DRIVE JOINT -->
-  <joint name="back_left_drive_joint" type="fixed">
+  <joint name="back_left_drive_joint" type="continuous">
     <parent link="back_left_knuckle"/>
     <child link="back_left_wheel"/>
     <origin xyz="${kwx} ${kwy} ${kwz}" rpy="${deg90} 0 ${deg180}"/>
+    <axis xyz="0 0 1"/>
   </joint>
   <!-- BACK RIGHT WHEEL POD -->
@@ -357,8 +363,9 @@
   </link>
   <!-- BACK RIGHT STEER JOINT -->
-  <joint name="back_right_steer_joint" type="fixed">
+  <joint name="back_right_steer_joint" type="continuous">
     <parent link="right_rocker"/>
     <child link="back_right_knuckle"/>
     <origin xyz="-${rkx} ${rky} ${rkz}" rpy="${deg90} 0 ${deg180}"/>
+    <axis xyz="0 0 -1"/>
   </joint>
   <!-- BACK RIGHT WHEEL -->
@@ -386,8 +393,9 @@
   </link>
   <!-- BACK RIGHT DRIVE JOINT -->
-  <joint name="back_right_drive_joint" type="fixed">
+  <joint name="back_right_drive_joint" type="continuous">
     <parent link="back_right_knuckle"/>
     <child link="back_right_wheel"/>
     <origin xyz="${kwx} ${kwy} ${kwz}" rpy="${deg90} 0 ${deg180}"/>
+    <axis xyz="0 0 1"/>
   </joint>
 </robot>

File: ros2_ws/src/lunabot_2425/description/ros2_control.xacro (robot description, xacro)
@@ -5,16 +5,9 @@
             <plugin>gz_ros2_control/GazeboSimSystem</plugin>
         </hardware>
-        <joint name="rear_left_drive_joint">
-            <command_interface name="velocity">
-                <param name="min">-10</param>
-                <param name="max">10</param>
-            </command_interface>
-            <state_interface name="velocity"/>
-            <state_interface name="position"/>
-        </joint>
-        <joint name="rear_right_drive_joint">
-            <command_interface name="velocity">
-                <param name="min">-10</param>
-                <param name="max">10</param>
+        <!-- front left -->
+        <joint name="front_left_steer_joint">
+            <command_interface name="position">
+                <param name="min">-95</param>
+                <param name="max">95</param>
             </command_interface>
             <state_interface name="velocity"/>
@@ -29,4 +22,13 @@
             <state_interface name="position"/>
         </joint>
+        <!-- front right -->
+        <joint name="front_right_steer_joint">
+            <command_interface name="position">
+                <param name="min">-95</param>
+                <param name="max">95</param>
+            </command_interface>
+            <state_interface name="velocity"/>
+            <state_interface name="position"/>
+        </joint>
         <joint name="front_right_drive_joint">
             <command_interface name="velocity">
@@ -37,5 +39,6 @@
             <state_interface name="position"/>
         </joint>
-        <joint name="rear_left_steer_joint">
+        <!-- back left -->
+        <joint name="back_left_steer_joint">
             <command_interface name="position">
                 <param name="min">-95</param>
@@ -45,5 +48,14 @@
             <state_interface name="position"/>
         </joint>
-        <joint name="rear_right_steer_joint">
+        <joint name="back_left_drive_joint">
+            <command_interface name="velocity">
+                <param name="min">-10</param>
+                <param name="max">10</param>
+            </command_interface>
+            <state_interface name="velocity"/>
+            <state_interface name="position"/>
+        </joint>
+        <!-- back right -->
+        <joint name="back_right_steer_joint">
             <command_interface name="position">
                 <param name="min">-95</param>
@@ -53,16 +65,8 @@
             <state_interface name="position"/>
         </joint>
-        <joint name="front_left_steer_joint">
-            <command_interface name="position">
-                <param name="min">-95</param>
-                <param name="max">95</param>
-            </command_interface>
-            <state_interface name="velocity"/>
-            <state_interface name="position"/>
-        </joint>
-        <joint name="front_right_steer_joint">
-            <command_interface name="position">
-                <param name="min">-95</param>
-                <param name="max">95</param>
+        <joint name="back_right_drive_joint">
+            <command_interface name="velocity">
+                <param name="min">-10</param>
+                <param name="max">10</param>
             </command_interface>
             <state_interface name="velocity"/>

Commit message: Robot can drive poorly

File: ros2_ws/src/lunabot_2425/description/robot_core.xacro (robot description, xacro)
@@ -367,5 +367,5 @@
     <child link="back_right_knuckle"/>
     <origin xyz="-${rkx} ${rky} ${rkz}" rpy="${deg90} 0 ${deg180}"/>
-    <axis xyz="0 0 -1"/>
+    <axis xyz="0 0 1"/>
   </joint>
   <!-- BACK RIGHT WHEEL -->
