Commit message: Fixed issue with one wheel driving inverted

File: ros2_ws/src/lunabot_2425/description/robot_core.xacro (robot description, xacro)
@@ -192,4 +192,5 @@
         <!-- <mesh filename="package://lunabot_2425/stl/wheel_mo.stl"/> -->
         <cylinder radius="${whee_rad}" length="${whee_len}"/>
+        <!-- <box size="${nuck_sx} ${nuck_sy} ${nuck_sz}"/> -->
       </geometry>
       <origin xyz="${whee_px} ${whee_py} ${whee_pz}" rpy="0 0 0"/>
@@ -208,4 +209,13 @@
       <inertia ixx="0.01" ixy="0" ixz="0" iyy="0.01" iyz="0" izz="0.01"/>
     </inertial>
+    <gazebo reference="front_left_wheel">
+      <mu1>0.9</mu1>
+      <mu2>0.9</mu2>
+      <kp>100000</kp>
+      <kd>1</kd>
+      <fdir1>1 0 0</fdir1>
+      <rolling_friction>0.02</rolling_friction>
+      <spinning_friction>0.02</spinning_friction>
+    </gazebo>
   </link>
   <!-- FRONT LEFT DRIVE JOINT -->
@@ -253,4 +263,5 @@
         <!-- <mesh filename="package://lunabot_2425/stl/wheel_mo.stl"/> -->
         <cylinder radius="${whee_rad}" length="${whee_len}"/>
+        <!-- <box size="${nuck_sx} ${nuck_sy} ${nuck_sz}"/> -->
       </geometry>
       <origin xyz="${whee_px} ${whee_py} ${whee_pz}" rpy="0 0 0"/>
@@ -269,4 +280,13 @@
       <inertia ixx="0.01" ixy="0" ixz="0" iyy="0.01" iyz="0" izz="0.01"/>
     </inertial>
+    <gazebo reference="front_right_wheel">
+      <mu1>0.9</mu1>
+      <mu2>0.9</mu2>
+      <kp>100000</kp>
+      <kd>1</kd>
+      <fdir1>1 0 0</fdir1>
+      <rolling_friction>0.02</rolling_friction>
+      <spinning_friction>0.02</spinning_friction>
+    </gazebo>
   </link>
   <!-- FRONT RIGHT DRIVE JOINT -->
@@ -314,4 +334,5 @@
         <!-- <mesh filename="package://lunabot_2425/stl/wheel_mo.stl"/> -->
         <cylinder radius="${whee_rad}" length="${whee_len}"/>
+        <!-- <box size="${nuck_sx} ${nuck_sy} ${nuck_sz}"/> -->
       </geometry>
       <origin xyz="${whee_px} ${whee_py} ${whee_pz}" rpy="0 0 0"/>
@@ -330,4 +351,13 @@
       <inertia ixx="0.01" ixy="0" ixz="0" iyy="0.01" iyz="0" izz="0.01"/>
     </inertial>
+    <gazebo reference="back_left_wheel">
+      <mu1>0.9</mu1>
+      <mu2>0.9</mu2>
+      <kp>100000</kp>
+      <kd>1</kd>
+      <fdir1>1 0 0</fdir1>
+      <rolling_friction>0.02</rolling_friction>
+      <spinning_friction>0.02</spinning_friction>
+    </gazebo>
   </link>
   <!-- BACK LEFT DRIVE JOINT -->
@@ -375,4 +405,5 @@
         <!-- <mesh filename="package://lunabot_2425/stl/wheel_mo.stl"/> -->
         <cylinder radius="${whee_rad}" length="${whee_len}"/>
+        <!-- <box size="${nuck_sx} ${nuck_sy} ${nuck_sz}"/> -->
       </geometry>
       <origin xyz="${whee_px} ${whee_py} ${whee_pz}" rpy="0 0 0"/>
@@ -391,4 +422,13 @@
       <inertia ixx="0.01" ixy="0" ixz="0" iyy="0.01" iyz="0" izz="0.01"/>
     </inertial>
+    <gazebo reference="back_right_wheel">
+      <mu1>0.9</mu1>
+      <mu2>0.9</mu2>
+      <kp>100000</kp>
+      <kd>1</kd>
+      <fdir1>1 0 0</fdir1>
+      <rolling_friction>0.02</rolling_friction>
+      <spinning_friction>0.02</spinning_friction>
+    </gazebo>
   </link>
   <!-- BACK RIGHT DRIVE JOINT -->
@@ -397,5 +437,5 @@
     <child link="back_right_wheel"/>
     <origin xyz="${kwx} ${kwy} ${kwz}" rpy="${deg90} 0 ${deg180}"/>
-    <axis xyz="0 0 1"/>
+    <axis xyz="0 0 -1"/>
   </joint>
 </robot>

Commit message: Rviz is gud, working on fixing other spawn issues and robot still drives funky

File: ros2_ws/src/lunabot_2425/description/robot_core.xacro (robot description, xacro)
@@ -191,6 +191,6 @@
       <geometry>
         <!-- <mesh filename="package://lunabot_2425/stl/wheel_mo.stl"/> -->
-        <cylinder radius="${whee_rad}" length="${whee_len}"/>
-        <!-- <box size="${nuck_sx} ${nuck_sy} ${nuck_sz}"/> -->
+        <!-- <cylinder radius="${whee_rad}" length="${whee_len}"/> -->
+        <box size="${nuck_sx} ${nuck_sy} ${nuck_sz}"/>
       </geometry>
       <origin xyz="${whee_px} ${whee_py} ${whee_pz}" rpy="0 0 0"/>
@@ -262,6 +262,6 @@
       <geometry>
         <!-- <mesh filename="package://lunabot_2425/stl/wheel_mo.stl"/> -->
-        <cylinder radius="${whee_rad}" length="${whee_len}"/>
-        <!-- <box size="${nuck_sx} ${nuck_sy} ${nuck_sz}"/> -->
+        <!-- <cylinder radius="${whee_rad}" length="${whee_len}"/> -->
+        <box size="${nuck_sx} ${nuck_sy} ${nuck_sz}"/>
       </geometry>
       <origin xyz="${whee_px} ${whee_py} ${whee_pz}" rpy="0 0 0"/>
@@ -333,6 +333,6 @@
       <geometry>
         <!-- <mesh filename="package://lunabot_2425/stl/wheel_mo.stl"/> -->
-        <cylinder radius="${whee_rad}" length="${whee_len}"/>
-        <!-- <box size="${nuck_sx} ${nuck_sy} ${nuck_sz}"/> -->
+        <!-- <cylinder radius="${whee_rad}" length="${whee_len}"/> -->
+        <box size="${nuck_sx} ${nuck_sy} ${nuck_sz}"/>
       </geometry>
       <origin xyz="${whee_px} ${whee_py} ${whee_pz}" rpy="0 0 0"/>
@@ -404,6 +404,6 @@
       <geometry>
         <!-- <mesh filename="package://lunabot_2425/stl/wheel_mo.stl"/> -->
-        <cylinder radius="${whee_rad}" length="${whee_len}"/>
-        <!-- <box size="${nuck_sx} ${nuck_sy} ${nuck_sz}"/> -->
+        <!-- <cylinder radius="${whee_rad}" length="${whee_len}"/> -->
+        <box size="${nuck_sx} ${nuck_sy} ${nuck_sz}"/>
       </geometry>
       <origin xyz="${whee_px} ${whee_py} ${whee_pz}" rpy="0 0 0"/>

Commit message: new apriltags and adjusted robot spawn loc

File: ros2_ws/src/lunabot_2425/description/robot_core.xacro (robot description, xacro)
@@ -191,4 +191,12 @@
       <geometry>
         <!-- <mesh filename="package://lunabot_2425/stl/wheel_mo.stl"/> -->
+        <cylinder radius="${whee_rad}" length="${whee_len}"/>
+        <!-- <box size="${nuck_sx} ${nuck_sy} ${nuck_sz}"/> -->
+      </geometry>
+      <origin xyz="${whee_px} ${whee_py} ${whee_pz}" rpy="0 0 0"/>
+    </visual>
+    <visual>
+      <geometry>
+        <!-- <mesh filename="package://lunabot_2425/stl/wheel_mo.stl"/> -->
         <!-- <cylinder radius="${whee_rad}" length="${whee_len}"/> -->
         <box size="${nuck_sx} ${nuck_sy} ${nuck_sz}"/>
@@ -262,4 +270,12 @@
       <geometry>
         <!-- <mesh filename="package://lunabot_2425/stl/wheel_mo.stl"/> -->
+        <cylinder radius="${whee_rad}" length="${whee_len}"/>
+        <!-- <box size="${nuck_sx} ${nuck_sy} ${nuck_sz}"/> -->
+      </geometry>
+      <origin xyz="${whee_px} ${whee_py} ${whee_pz}" rpy="0 0 0"/>
+    </visual>
+    <visual>
+      <geometry>
+        <!-- <mesh filename="package://lunabot_2425/stl/wheel_mo.stl"/> -->
         <!-- <cylinder radius="${whee_rad}" length="${whee_len}"/> -->
         <box size="${nuck_sx} ${nuck_sy} ${nuck_sz}"/>
@@ -333,4 +349,12 @@
       <geometry>
         <!-- <mesh filename="package://lunabot_2425/stl/wheel_mo.stl"/> -->
+        <cylinder radius="${whee_rad}" length="${whee_len}"/>
+        <!-- <box size="${nuck_sx} ${nuck_sy} ${nuck_sz}"/> -->
+      </geometry>
+      <origin xyz="${whee_px} ${whee_py} ${whee_pz}" rpy="0 0 0"/>
+    </visual>
+    <visual>
+      <geometry>
+        <!-- <mesh filename="package://lunabot_2425/stl/wheel_mo.stl"/> -->
         <!-- <cylinder radius="${whee_rad}" length="${whee_len}"/> -->
         <box size="${nuck_sx} ${nuck_sy} ${nuck_sz}"/>
@@ -404,4 +428,12 @@
       <geometry>
         <!-- <mesh filename="package://lunabot_2425/stl/wheel_mo.stl"/> -->
+        <cylinder radius="${whee_rad}" length="${whee_len}"/>
+        <!-- <box size="${nuck_sx} ${nuck_sy} ${nuck_sz}"/> -->
+      </geometry>
+      <origin xyz="${whee_px} ${whee_py} ${whee_pz}" rpy="0 0 0"/>
+    </visual>
+    <visual>
+      <geometry>
+        <!-- <mesh filename="package://lunabot_2425/stl/wheel_mo.stl"/> -->
         <!-- <cylinder radius="${whee_rad}" length="${whee_len}"/> -->
         <box size="${nuck_sx} ${nuck_sy} ${nuck_sz}"/>
