Commit message: Added 4 visual cameras need to think through frames soon

File: ros2_ws/src/lunabot_2425/description/camera.xacro (robot description, xacro)
@@ -1,44 +1,63 @@
 <?xml version="1.0"?>
-<robot xmlns:xacro="http://www.ros.org/wiki/xacro" name="robot">
-    <joint name="camera_joint" type="fixed">
-        <parent link="base_link" />
-        <child link="camera_link" />
-        <origin xyz="0.275 0.12 1.17" rpy="0 0.6 0" />
+<robot xmlns:xacro="http://www.ros.org/wiki/xacro">
+  <!-- Macro: generic camera with parametric pose and naming -->
+  <xacro:macro name="camera_module" params="
+      parent_link
+      cam_name:=camera
+      xyz:='0 0 0'
+      rpy:='0 0 0'
+      radius:=0.05
+      length:=0.04
+      fov:=1.089
+      width:=640
+      height:=480
+      clip_near:=0.05
+      clip_far:=8.0
+  ">
+    <!-- BASE JOINT -->
+    <joint name="${cam_name}_joint" type="fixed">
+      <parent link="${parent_link}"/>
+      <child link="${cam_name}_link"/>
+      <origin xyz="${xyz}" rpy="${rpy}"/>
     </joint>
-    <link name="camera_link">
-        <visual>
-            <geometry>
-                <cylinder radius="0.05" length="0.04" />
-                <material name="green" />
-            </geometry>
-            <material name="green" />
-        </visual>
+    <!-- CAMERA BODY LINK -->
+    <link name="${cam_name}_link">
+      <visual>
+        <geometry>
+          <cylinder radius="${radius}" length="${length}"/>
+        </geometry>
+        <origin xyz="0 0 0" rpy="0 -1.57079632679 0"/>
+        <material name="green"/>
+      </visual>
     </link>
-    <joint name="camera_optical_joint" type="fixed">
-        <parent link="camera_link" />
-        <child link="camera_link_optical" />
-        <origin xyz="0 0 0" rpy="-1.57079632679 0 -1.57079632679" />
+    <!-- OPTICAL FRAME -->
+    <joint name="${cam_name}_optical_joint" type="fixed">
+      <parent link="${cam_name}_link"/>
+      <child link="${cam_name}_link_optical"/>
+      <origin xyz="0 0 0" rpy="-1.57079632679 0 -1.57079632679"/>
     </joint>
-    <link name="camera_link_optical"></link>
-    <gazebo reference="camera_link">
-        <sensor name="camera" type="camera">
-            <camera>
-                <camera_info_topic>camera/camera_info</camera_info_topic>
-                <horizontal_fov>1.089</horizontal_fov>
-                <image>
-                    <format>R8G8B8</format>
-                    <width>640</width>
-                    <height>480</height>
-                </image>
-                <clip>
-                    <near>0.05</near>
-                    <far>8.0</far>
-                </clip>
-            </camera>
-            <visualize>true</visualize>
-            <update_rate>15</update_rate>
-            <topic>camera/image_raw</topic>
-            <gz_frame_id>camera_link_optical</gz_frame_id>
-        </sensor>
+    <link name="${cam_name}_link_optical"/>
+    <!-- GAZEBO SENSOR -->
+    <gazebo reference="${cam_name}_link">
+      <sensor name="${cam_name}" type="camera">
+        <camera>
+          <camera_info_topic>${cam_name}/camera_info</camera_info_topic>
+          <horizontal_fov>${fov}</horizontal_fov>
+          <image>
+            <format>R8G8B8</format>
+            <width>${width}</width>
+            <height>${height}</height>
+          </image>
+          <clip>
+            <near>${clip_near}</near>
+            <far>${clip_far}</far>
+          </clip>
+        </camera>
+        <visualize>true</visualize>
+        <update_rate>15</update_rate>
+        <topic>${cam_name}/image_raw</topic>
+        <gz_frame_id>${cam_name}_link_optical</gz_frame_id>
+      </sensor>
     </gazebo>
+  </xacro:macro>
 </robot>

File: ros2_ws/src/lunabot_2425/description/robot.urdf.xacro (robot description, xacro)
@@ -8,3 +8,24 @@
     <xacro:include filename="realsense_d455_macro.xacro" />
     <xacro:realsense_camera parent_link="base_link" />
+    <xacro:include filename="camera.xacro" />
+    <xacro:camera_module
+    cam_name="front_left_camera"
+    parent_link="front_left_knuckle"
+    xyz="0 0 0.25"
+    rpy="0 0 0"/>
+    <xacro:camera_module
+    cam_name="front_right_camera"
+    parent_link="front_right_knuckle"
+    xyz="0 0 0.25"
+    rpy="0 0 1.570796"/>
+    <xacro:camera_module
+    cam_name="back_left_camera"
+    parent_link="back_left_knuckle"
+    xyz="-0 0 0.25"
+    rpy="0 0 1.570796"/>
+    <xacro:camera_module
+    cam_name="back_right_camera"
+    parent_link="back_right_knuckle"
+    xyz="-0 0 0.25"
+    rpy="0 0 0"/>
 </robot>

Commit message: Add Jetson hardware / camera smoke test workflow
- Fiducial: single-cam hardware YAML, hardware test params, localizer tweaks
- lunabot_2425: hardware_smoke.launch.py, hardware_bringup updates
- luna_mapping: EKF global config, odom relay, depth crater detector, launch wiring
- luna_nav: mission and Nav2 config updates
- Docs: HARDWARE_SMOKE_TEST.md; build_workspace helper
- Submodule luna_ros2_worlds: arena and crater model updates

Made-with: Cursor

File: ros2_ws/src/lunabot_2425/description/camera.xacro (robot description, xacro)
@@ -9,5 +9,5 @@
       radius:=0.05
       length:=0.04
-      fov:=1.869
+      fov:=2.094
       width:=1280
       height:=720

File: ros2_ws/src/lunabot_2425/description/realsense_d455_macro.xacro (robot description, xacro)
@@ -26,5 +26,5 @@
       <parent link="${parent_link}"/>
       <child link="depth_camera_link"/>
-      <origin xyz="0.3 0.1 0.65" rpy="0 0.49 0"/>
+      <origin xyz="0.3 0.1 0.65" rpy="0 0.262 0"/>
     </joint>
     <!-- ===== Optical frames for ROS conventions ===== -->
