Commit message: set up URDF stuff with hardware iface. builds but throws param error on launch

File: ros2_ws/src/lunabot_2425/description/robot.urdf.xacro (robot description, xacro)
@@ -1,7 +1,14 @@
 <?xml version="1.0"?>
 <robot xmlns:xacro="http://www.ros.org/wiki/xacro" name="robot">
+    <xacro:arg name="use_sim" default="true"/>
     <xacro:include filename="robot_core.xacro" />
     <!-- <xacro:include filename="gz_control.xacro" /> -->
+    <!-- Select hardware interface based on use_sim arg -->
+    <xacro:if value="$(arg use_sim)">
     <xacro:include filename="ros2_control.xacro" />
+    </xacro:if>
+    <xacro:unless value="$(arg use_sim)">
+    <xacro:include filename="ros2_control_hw.xacro" />
+    </xacro:unless>
     <!-- <xacro:include filename="camera.xacro" /> -->
     <!-- <xacro:include filename="depth_camera.xacro" /> -->

File: ros2_ws/src/lunabot_2425/description/robot_core.xacro (robot description, xacro)
@@ -180,5 +180,6 @@
   </link>
   <!-- FRONT LEFT STEER JOINT -->
-  <joint name="front_left_steer_joint" type="continuous">
+  <joint name="front_left_steer_joint" type="revolute">
+    <limit lower="-1.658" upper="1.658" effort="10.0" velocity="2.0"/>
     <parent link="left_rocker"/>
     <child link="front_left_knuckle"/>
@@ -259,5 +260,6 @@
   </link>
   <!-- FRONT RIGHT STEER JOINT -->
-  <joint name="front_right_steer_joint" type="continuous">
+  <joint name="front_right_steer_joint" type="revolute">
+    <limit lower="-1.658" upper="1.658" effort="10.0" velocity="2.0"/>
     <parent link="right_rocker"/>
     <child link="front_right_knuckle"/>
@@ -338,5 +340,6 @@
   </link>
   <!-- BACK LEFT STEER JOINT -->
-  <joint name="back_left_steer_joint" type="continuous">
+  <joint name="back_left_steer_joint" type="revolute">
+    <limit lower="-1.658" upper="1.658" effort="10.0" velocity="2.0"/>
     <parent link="left_rocker"/>
     <child link="back_left_knuckle"/>
@@ -417,5 +420,6 @@
   </link>
   <!-- BACK RIGHT STEER JOINT -->
-  <joint name="back_right_steer_joint" type="continuous">
+  <joint name="back_right_steer_joint" type="revolute">
+    <limit lower="-1.658" upper="1.658" effort="10.0" velocity="2.0"/>
     <parent link="right_rocker"/>
     <child link="back_right_knuckle"/>
