Commit message: All dept/color sensors work minus the missing pointclpud

File: ros2_ws/src/lunabot_2425/description/realsense_d455_macro.xacro (robot description, xacro)
@@ -2,5 +2,4 @@
 <robot xmlns:xacro="http://www.ros.org/wiki/xacro">
   <xacro:macro name="realsense_camera" params="parent_link">
-    <!-- Camera link -->
     <link name="camera_link">
       <visual>
@@ -19,5 +18,6 @@
       <inertial>
         <mass value="0.2"/>
-        <inertia ixx="0.0001" ixy="0.0" ixz="0.0" iyy="0.0001" iyz="0.0" izz="0.0001"/>
+        <inertia ixx="0.0001" ixy="0" ixz="0"
+                iyy="0.0001" iyz="0" izz="0.0001"/>
       </inertial>
     </link>
@@ -26,35 +26,16 @@
       <parent link="${parent_link}"/>
       <child link="camera_link"/>
-      <origin xyz="0.1 0 0.2" rpy="0 0 0"/>
+      <origin xyz="0.1 0 0.65" rpy="0 1 0"/>
     </joint>
-    <!-- RGB Camera -->
+    <!-- ======================================================= -->
+    <!-- ================= GAZEBO HARMONIC SENSORS ============= -->
+    <!-- ======================================================= -->
     <gazebo reference="camera_link">
-      <sensor type="camera" name="d455_rgb_camera">
-        <pose>0 0 0 0 0 0</pose>
-        <camera>
-          <horizontal_fov>1.0467</horizontal_fov> <!-- 60 degrees -->
-          <image>
-            <width>1280</width>
-            <height>720</height>
-            <format>R8G8B8</format>
-          </image>
-          <clip>
-            <near>0.1</near>
-            <far>10.0</far>
-          </clip>
-        </camera>
-        <plugin name="gazebo_ros_camera_rgb" filename="libgazebo_ros_camera.so">
-          <ros>
-            <namespace>/camera/rgb</namespace>
-            <remapping>image:=image_raw</remapping>
-          </ros>
-          <camera_name>d455_rgb</camera_name>
-          <frame_name>camera_link</frame_name>
-        </plugin>
-      </sensor>
-    </gazebo>
-    <!-- Depth Camera -->
-    <gazebo reference="camera_link">
-      <sensor type="depth" name="d455_depth_camera">
+      <!-- ================= RGB CAMERA ================= -->
+      <sensor name="d455_rgb_camera" type="camera">
+        <!-- Internal Gazebo topic -->
+        <topic>/sim/camera/rgb/image</topic>
+        <always_on>true</always_on>
+        <update_rate>30</update_rate>
         <pose>0 0 0 0 0 0</pose>
         <camera>
@@ -65,17 +46,32 @@
             <format>R8G8B8</format>
           </image>
-          <clip>
-            <near>0.1</near>
-            <far>10.0</far>
-          </clip>
+          <clip><near>0.1</near><far>20.0</far></clip>
+          <render_engine>ogre</render_engine>
         </camera>
-        <plugin name="gazebo_ros_depth_camera" filename="libgazebo_ros_depth_camera.so">
-          <ros>
-            <namespace>/camera/depth</namespace>
-            <remapping>depth/image_raw:=depth_image</remapping>
-          </ros>
-          <camera_name>d455_depth</camera_name>
-          <frame_name>camera_link</frame_name>
-        </plugin>
+        <frame>camera_color_optical_frame</frame>
+      </sensor>
+      <!-- ================= DEPTH CAMERA ================= -->
+      <sensor name="d455_depth_camera" type="depth">
+        <!-- Internal Gazebo topics -->
+        <topic>/sim/camera/depth/image</topic>
+        <always_on>true</always_on>
+        <update_rate>30</update_rate>
+        <pose>0 0 0 0 0 0</pose>
+        <camera>
+          <horizontal_fov>1.0467</horizontal_fov>
+          <image>
+            <width>1280</width>
+            <height>720</height>
+            <format>R8G8B8</format> <!-- Depth format for bridge -->
+          </image>
+          <clip><near>0.1</near><far>20.0</far></clip>
+          <render_engine>ogre</render_engine>
+        </camera>
+        <!-- Optional: packed depth for pointcloud conversion -->
+        <publisher>
+          <topic>/sim/camera/depth/image_packed</topic>
+          <type>pointcloud_packed</type>
+        </publisher>
+        <frame>camera_depth_optical_frame</frame>
       </sensor>
     </gazebo>

Commit message: fixed launch file

File: ros2_ws/src/lunabot_2425/description/realsense_d455_macro.xacro (robot description, xacro)
@@ -26,5 +26,5 @@
       <parent link="${parent_link}"/>
       <child link="camera_link"/>
-      <origin xyz="0.1 0 0.65" rpy="0 1 0"/>
+      <origin xyz="0.3 0.1 0.65" rpy="0 1 0"/>
     </joint>
     <!-- ======================================================= -->

Commit message: reverted Luis merge of nav2, something went wrong?

File: ros2_ws/src/lunabot_2425/description/realsense_d455_macro.xacro (robot description, xacro)
@@ -2,5 +2,5 @@
 <robot xmlns:xacro="http://www.ros.org/wiki/xacro">
   <xacro:macro name="realsense_camera" params="parent_link">
-    <link name="camera_link">
+    <link name="depth_camera_link">
       <visual>
         <geometry>
@@ -23,7 +23,7 @@
     </link>
     <!-- Fixed joint connecting camera to robot -->
-    <joint name="camera_joint" type="fixed">
+    <joint name="depth_camera_joint" type="fixed">
       <parent link="${parent_link}"/>
-      <child link="camera_link"/>
+      <child link="depth_camera_link"/>
       <origin xyz="0.3 0.1 0.65" rpy="0 1 0"/>
     </joint>
@@ -31,5 +31,5 @@
     <!-- ================= GAZEBO HARMONIC SENSORS ============= -->
     <!-- ======================================================= -->
-    <gazebo reference="camera_link">
+    <gazebo reference="depth_camera_link">
       <!-- ================= RGB CAMERA ================= -->
       <sensor name="d455_rgb_camera" type="camera">

Commit message: Add RTAB-Map + Nav2 costmap integration with depth camera
- Integrated RTAB-Map SLAM for occupancy grid generation from RealSense D455
- Added Nav2 navigation stack with depth-based costmaps
- Created depth-to-laserscan and depth-to-pointcloud converters
- Added camera_info and image frame_id fixers for Gazebo compatibility
- Updated URDF with proper optical frames for cameras
- Added static TF transforms for odom->base_link and camera frames
- Created comprehensive launch file: rtabmap_nav2_sim.launch.py
- Updated topic names to match existing conventions (/camera/camera/...)
- Added Nav2 configuration for depth-based obstacle detection
- Created RViz config and documentation files

File: ros2_ws/src/lunabot_2425/description/realsense_d455_macro.xacro (robot description, xacro)
@@ -27,4 +27,27 @@
       <child link="depth_camera_link"/>
       <origin xyz="0.3 0.1 0.65" rpy="0 1 0"/>
+    </joint>
+    <!-- ===== Optical frames for ROS conventions ===== -->
+    <!-- Color optical frame (rotated for camera coordinate system: Z forward, X right, Y down) -->
+    <link name="camera_color_optical_frame"/>
+    <joint name="camera_color_optical_joint" type="fixed">
+      <parent link="depth_camera_link"/>
+      <child link="camera_color_optical_frame"/>
+      <!-- Rotation: -90 deg roll, 0 pitch, -90 deg yaw transforms robot frame to optical frame -->
+      <origin xyz="0 0 0" rpy="-1.5708 0 -1.5708"/>
+    </joint>
+    <!-- Depth optical frame (same orientation as color for aligned depth) -->
+    <link name="camera_depth_optical_frame"/>
+    <joint name="camera_depth_optical_joint" type="fixed">
+      <parent link="depth_camera_link"/>
+      <child link="camera_depth_optical_frame"/>
+      <origin xyz="0 0 0" rpy="-1.5708 0 -1.5708"/>
+    </joint>
+    <!-- Camera link (standard ROS naming convention) -->
+    <link name="camera_link"/>
+    <joint name="camera_link_joint" type="fixed">
+      <parent link="depth_camera_link"/>
+      <child link="camera_link"/>
+      <origin xyz="0 0 0" rpy="0 0 0"/>
     </joint>
     <!-- ======================================================= -->

Commit message: Sim: merge RTAB-Map+Nav2 into gz_bringup (single terminal); add hardware bringup and docs
- gz_bringup: launch_mapping (default true) starts RTAB-Map/Nav2 after ~18s
- lunabot_2425: hardware_bringup.launch.py (RealSense D455 + 4x Nexigo N980P)
- luna_mapping: rtabmap_nav2_hardware.launch.py, sim launch accepts sim:=false for hardware
- Nav2: static map only; RTAB-Map grid tuning (MaxGroundHeight, RangeMin, DepthDecimation)
- depth_fov_filter: static mask (mask_regions) instead of FOV crop
- docs/HARDWARE.md, README and LAUNCH_COMMANDS updated; Dockerfile.jetson added

File: ros2_ws/src/lunabot_2425/description/realsense_d455_macro.xacro (robot description, xacro)
@@ -26,5 +26,5 @@
       <parent link="${parent_link}"/>
       <child link="depth_camera_link"/>
-      <origin xyz="0.3 0.1 0.65" rpy="0 1 0"/>
+      <origin xyz="0.3 0.1 0.65" rpy="0 0.49 0"/>
     </joint>
     <!-- ===== Optical frames for ROS conventions ===== -->
@@ -76,5 +76,4 @@
       <!-- ================= DEPTH CAMERA ================= -->
       <sensor name="d455_depth_camera" type="depth">
-        <!-- Internal Gazebo topics -->
         <topic>/sim/camera/depth/image</topic>
         <always_on>true</always_on>
@@ -86,5 +85,5 @@
             <width>1280</width>
             <height>720</height>
-            <format>R8G8B8</format> <!-- Depth format for bridge -->
+            <format>R8G8B8</format>
           </image>
           <clip><near>0.1</near><far>20.0</far></clip>

Commit message: Bring forward working stack from fiducial_shit onto clean master base
Cherry-picked final state of key packages:
- fiducial_localizer: multi-camera ArUco detection with ParameterValue fix
- luna_mapping: RTAB-Map + Nav2 sim launch, frame fixers, height filter
- luna_nav: Nav2 params, zone_publisher node, config files
- lunabot_2425: gz_bringup with arena selection, hardware_bringup
- luna_control, depth_to_pointcloud, run_ros_image.sh updates

Made-with: Cursor

File: ros2_ws/src/lunabot_2425/description/realsense_d455_macro.xacro (robot description, xacro)
@@ -2,5 +2,5 @@
 <robot xmlns:xacro="http://www.ros.org/wiki/xacro">
   <xacro:macro name="realsense_camera" params="parent_link">
-    <link name="camera_link">
+    <link name="depth_camera_link">
       <visual>
         <geometry>
@@ -23,16 +23,38 @@
     </link>
     <!-- Fixed joint connecting camera to robot -->
-    <joint name="camera_joint" type="fixed">
+    <joint name="depth_camera_joint" type="fixed">
       <parent link="${parent_link}"/>
+      <child link="depth_camera_link"/>
+      <origin xyz="0.3 0.1 0.65" rpy="0 0.49 0"/>
+    </joint>
+    <!-- ===== Optical frames for ROS conventions ===== -->
+    <!-- Color optical frame (rotated for camera coordinate system: Z forward, X right, Y down) -->
+    <link name="camera_color_optical_frame"/>
+    <joint name="camera_color_optical_joint" type="fixed">
+      <parent link="depth_camera_link"/>
+      <child link="camera_color_optical_frame"/>
+      <!-- Rotation: -90 deg roll, 0 pitch, -90 deg yaw transforms robot frame to optical frame -->
+      <origin xyz="0 0 0" rpy="-1.5708 0 -1.5708"/>
+    </joint>
+    <!-- Depth optical frame (same orientation as color for aligned depth) -->
+    <link name="camera_depth_optical_frame"/>
+    <joint name="camera_depth_optical_joint" type="fixed">
+      <parent link="depth_camera_link"/>
+      <child link="camera_depth_optical_frame"/>
+      <origin xyz="0 0 0" rpy="-1.5708 0 -1.5708"/>
+    </joint>
+    <!-- Camera link (standard ROS naming convention) -->
+    <link name="camera_link"/>
+    <joint name="camera_link_joint" type="fixed">
+      <parent link="depth_camera_link"/>
       <child link="camera_link"/>
-      <origin xyz="0.3 0.1 0.65" rpy="0 1 0"/>
+      <origin xyz="0 0 0" rpy="0 0 0"/>
     </joint>
     <!-- ======================================================= -->
     <!-- ================= GAZEBO HARMONIC SENSORS ============= -->
     <!-- ======================================================= -->
-    <gazebo reference="camera_link">
+    <gazebo reference="depth_camera_link">
       <!-- ================= RGB CAMERA ================= -->
       <sensor name="d455_rgb_camera" type="camera">
-        <!-- Internal Gazebo topic -->
         <topic>/sim/camera/rgb/image</topic>
         <always_on>true</always_on>
@@ -40,5 +62,6 @@
         <pose>0 0 0 0 0 0</pose>
         <camera>
-          <horizontal_fov>1.0467</horizontal_fov>
+          <!-- D455 RGB: 86deg H-FOV = 1.5009 rad -->
+          <horizontal_fov>1.5009</horizontal_fov>
           <image>
             <width>1280</width>
@@ -46,5 +69,5 @@
             <format>R8G8B8</format>
           </image>
-          <clip><near>0.1</near><far>20.0</far></clip>
+          <clip><near>0.1</near><far>10.0</far></clip>
           <render_engine>ogre</render_engine>
         </camera>
@@ -53,5 +76,4 @@
       <!-- ================= DEPTH CAMERA ================= -->
       <sensor name="d455_depth_camera" type="depth">
-        <!-- Internal Gazebo topics -->
         <topic>/sim/camera/depth/image</topic>
         <always_on>true</always_on>
@@ -59,11 +81,12 @@
         <pose>0 0 0 0 0 0</pose>
         <camera>
-          <horizontal_fov>1.0467</horizontal_fov>
+          <!-- D455 Depth: 86deg H-FOV = 1.5009 rad -->
+          <horizontal_fov>1.5009</horizontal_fov>
           <image>
             <width>1280</width>
             <height>720</height>
-            <format>R8G8B8</format> <!-- Depth format for bridge -->
+            <format>R8G8B8</format>
           </image>
-          <clip><near>0.1</near><far>20.0</far></clip>
+          <clip><near>0.2</near><far>10.0</far></clip>
           <render_engine>ogre</render_engine>
         </camera>

Commit message: removed more semicolons from URDF

File: ros2_ws/src/lunabot_2425/description/realsense_d455_macro.xacro (robot description, xacro)
@@ -62,5 +62,5 @@
         <pose>0 0 0 0 0 0</pose>
         <camera>
-          <!-- D455 RGB: 86deg H-FOV = 1.5009 rad -->
+          <!-- D455 RGB  86deg H-FOV = 1.5009 rad -->
           <horizontal_fov>1.5009</horizontal_fov>
           <image>
@@ -81,5 +81,5 @@
         <pose>0 0 0 0 0 0</pose>
         <camera>
-          <!-- D455 Depth: 86deg H-FOV = 1.5009 rad -->
+          <!-- D455 Depth 86deg H-FOV = 1.5009 rad -->
           <horizontal_fov>1.5009</horizontal_fov>
           <image>

File: ros2_ws/src/lunabot_2425/description/robot.urdf.xacro (robot description, xacro)
@@ -3,5 +3,5 @@
     <xacro:arg name="use_sim" default="true"/>
     <xacro:include filename="robot_core.xacro" />
-    <!-- <xacro:include filename="gz_control.xacro" /> -->
+    <!-- <xacro include filename="gz_control.xacro" /> -->
     <!-- Select hardware interface based on use_sim arg -->
     <xacro:if value="$(arg use_sim)">
@@ -11,6 +11,6 @@
     <xacro:include filename="ros2_control_hw.xacro" />
     </xacro:unless>
-    <!-- <xacro:include filename="camera.xacro" /> -->
-    <!-- <xacro:include filename="depth_camera.xacro" /> -->
+    <!-- <xacro include filename="camera.xacro" /> -->
+    <!-- <xacro include filename="depth_camera.xacro" /> -->
     <xacro:include filename="realsense_d455_macro.xacro" />
     <xacro:realsense_camera parent_link="base_link" />

File: ros2_ws/src/lunabot_2425/description/robot_core.xacro (robot description, xacro)
@@ -72,5 +72,5 @@
     <visual>
       <geometry>
-        <!-- <mesh filename="package://lunabot_2425/stl/bucket_mo.stl"/> -->
+        <!-- <mesh filename="package //lunabot_2425/stl/bucket_mo.stl"/> -->
         <box size="${buck_sx} ${buck_sy} ${buck_sz}"/>
       </geometry>
@@ -80,5 +80,5 @@
     <collision>
       <geometry>
-        <!-- <mesh filename="package://lunabot_2425/stl/bucket_mo.stl"/> -->
+        <!-- <mesh filename="package //lunabot_2425/stl/bucket_mo.stl"/> -->
         <box size="${buck_sx} ${buck_sy} ${buck_sz}"/>
       </geometry>
@@ -101,5 +101,5 @@
     <visual>
       <geometry>
-        <!-- <mesh filename="package://lunabot_2425/stl/left_rocker_mo.stl"/> -->
+        <!-- <mesh filename="package //lunabot_2425/stl/left_rocker_mo.stl"/> -->
         <cylinder radius="${rock_rad}" length="${rock_len}"/>
       </geometry>
@@ -109,5 +109,5 @@
     <collision>
       <geometry>
-        <!-- <mesh filename="package://lunabot_2425/stl/left_rocker_mo.stl"/> -->
+        <!-- <mesh filename="package //lunabot_2425/stl/left_rocker_mo.stl"/> -->
         <cylinder radius="${rock_rad}" length="${rock_len}"/>
       </geometry>
@@ -130,5 +130,5 @@
     <visual>
       <geometry>
-        <!-- <mesh filename="package://lunabot_2425/stl/right_rocker_mo.stl"/> -->
+        <!-- <mesh filename="package //lunabot_2425/stl/right_rocker_mo.stl"/> -->
         <cylinder radius="${rock_rad}" length="${rock_len}"/>
       </geometry>
@@ -138,5 +138,5 @@
     <collision>
       <geometry>
-        <!-- <mesh filename="package://lunabot_2425/stl/right_rocker_mo.stl"/> -->
+        <!-- <mesh filename="package //lunabot_2425/stl/right_rocker_mo.stl"/> -->
         <cylinder radius="${rock_rad}" length="${rock_len}"/>
       </geometry>
@@ -160,5 +160,5 @@
     <visual>
       <geometry>
-        <!-- <mesh filename="package://lunabot_2425/stl/knuckle_mo.stl"/> -->
+        <!-- <mesh filename="package //lunabot_2425/stl/knuckle_mo.stl"/> -->
         <box size="${nuck_sx} ${nuck_sy} ${nuck_sz}"/>
       </geometry>
@@ -168,5 +168,5 @@
     <collision>
       <geometry>
-        <!-- <mesh filename="package://lunabot_2425/stl/knuckle_mo.stl"/> -->
+        <!-- <mesh filename="package //lunabot_2425/stl/knuckle_mo.stl"/> -->
         <box size="${nuck_sx} ${nuck_sy} ${nuck_sz}"/>
       </geometry>
@@ -191,5 +191,5 @@
     <visual>
       <geometry>
-        <!-- <mesh filename="package://lunabot_2425/stl/wheel_mo.stl"/> -->
+        <!-- <mesh filename="package //lunabot_2425/stl/wheel_mo.stl"/> -->
         <cylinder radius="${whee_rad}" length="${whee_len}"/>
         <!-- <box size="${nuck_sx} ${nuck_sy} ${nuck_sz}"/> -->
@@ -199,5 +199,5 @@
     <visual>
       <geometry>
-        <!-- <mesh filename="package://lunabot_2425/stl/wheel_mo.stl"/> -->
+        <!-- <mesh filename="package //lunabot_2425/stl/wheel_mo.stl"/> -->
         <!-- <cylinder radius="${whee_rad}" length="${whee_len}"/> -->
         <box size="${nuck_sx} ${nuck_sy} ${nuck_sz}"/>
@@ -208,5 +208,5 @@
     <collision>
       <geometry>
-        <!-- <mesh filename="package://lunabot_2425/stl/wheel_mo.stl"/> -->
+        <!-- <mesh filename="package //lunabot_2425/stl/wheel_mo.stl"/> -->
         <cylinder radius="${whee_rad}" length="${whee_len}"/>
       </geometry>
@@ -240,5 +240,5 @@
     <visual>
       <geometry>
-        <!-- <mesh filename="package://lunabot_2425/stl/knuckle_mo.stl"/> -->
+        <!-- <mesh filename="package //lunabot_2425/stl/knuckle_mo.stl"/> -->
         <box size="${nuck_sx} ${nuck_sy} ${nuck_sz}"/>
       </geometry>
@@ -248,5 +248,5 @@
     <collision>
       <geometry>
-        <!-- <mesh filename="package://lunabot_2425/stl/knuckle_mo.stl"/> -->
+        <!-- <mesh filename="package //lunabot_2425/stl/knuckle_mo.stl"/> -->
         <box size="${nuck_sx} ${nuck_sy} ${nuck_sz}"/>
       </geometry>
@@ -271,5 +271,5 @@
     <visual>
       <geometry>
-        <!-- <mesh filename="package://lunabot_2425/stl/wheel_mo.stl"/> -->
+        <!-- <mesh filename="package //lunabot_2425/stl/wheel_mo.stl"/> -->
         <cylinder radius="${whee_rad}" length="${whee_len}"/>
         <!-- <box size="${nuck_sx} ${nuck_sy} ${nuck_sz}"/> -->
@@ -279,5 +279,5 @@
     <visual>
       <geometry>
-        <!-- <mesh filename="package://lunabot_2425/stl/wheel_mo.stl"/> -->
+        <!-- <mesh filename="package //lunabot_2425/stl/wheel_mo.stl"/> -->
         <!-- <cylinder radius="${whee_rad}" length="${whee_len}"/> -->
         <box size="${nuck_sx} ${nuck_sy} ${nuck_sz}"/>
@@ -288,5 +288,5 @@
     <collision>
       <geometry>
-        <!-- <mesh filename="package://lunabot_2425/stl/wheel_mo.stl"/> -->
+        <!-- <mesh filename="package //lunabot_2425/stl/wheel_mo.stl"/> -->
         <cylinder radius="${whee_rad}" length="${whee_len}"/>
       </geometry>
@@ -320,5 +320,5 @@
     <visual>
       <geometry>
-        <!-- <mesh filename="package://lunabot_2425/stl/knuckle_mo.stl"/> -->
+        <!-- <mesh filename="package //lunabot_2425/stl/knuckle_mo.stl"/> -->
         <box size="${nuck_sx} ${nuck_sy} ${nuck_sz}"/>
       </geometry>
@@ -328,5 +328,5 @@
     <collision>
       <geometry>
-        <!-- <mesh filename="package://lunabot_2425/stl/knuckle_mo.stl"/> -->
+        <!-- <mesh filename="package //lunabot_2425/stl/knuckle_mo.stl"/> -->
         <box size="${nuck_sx} ${nuck_sy} ${nuck_sz}"/>
       </geometry>
@@ -351,5 +351,5 @@
     <visual>
       <geometry>
-        <!-- <mesh filename="package://lunabot_2425/stl/wheel_mo.stl"/> -->
+        <!-- <mesh filename="package //lunabot_2425/stl/wheel_mo.stl"/> -->
         <cylinder radius="${whee_rad}" length="${whee_len}"/>
         <!-- <box size="${nuck_sx} ${nuck_sy} ${nuck_sz}"/> -->
@@ -359,5 +359,5 @@
     <visual>
       <geometry>
-        <!-- <mesh filename="package://lunabot_2425/stl/wheel_mo.stl"/> -->
+        <!-- <mesh filename="package //lunabot_2425/stl/wheel_mo.stl"/> -->
         <!-- <cylinder radius="${whee_rad}" length="${whee_len}"/> -->
         <box size="${nuck_sx} ${nuck_sy} ${nuck_sz}"/>
@@ -368,5 +368,5 @@
     <collision>
       <geometry>
-        <!-- <mesh filename="package://lunabot_2425/stl/wheel_mo.stl"/> -->
+        <!-- <mesh filename="package //lunabot_2425/stl/wheel_mo.stl"/> -->
         <cylinder radius="${whee_rad}" length="${whee_len}"/>
       </geometry>
@@ -400,5 +400,5 @@
     <visual>
       <geometry>
-        <!-- <mesh filename="package://lunabot_2425/stl/knuckle_mo.stl"/> -->
+        <!-- <mesh filename="package //lunabot_2425/stl/knuckle_mo.stl"/> -->
         <box size="${nuck_sx} ${nuck_sy} ${nuck_sz}"/>
       </geometry>
@@ -408,5 +408,5 @@
     <collision>
       <geometry>
-        <!-- <mesh filename="package://lunabot_2425/stl/knuckle_mo.stl"/> -->
+        <!-- <mesh filename="package //lunabot_2425/stl/knuckle_mo.stl"/> -->
         <box size="${nuck_sx} ${nuck_sy} ${nuck_sz}"/>
       </geometry>
@@ -431,5 +431,5 @@
     <visual>
       <geometry>
-        <!-- <mesh filename="package://lunabot_2425/stl/wheel_mo.stl"/> -->
+        <!-- <mesh filename="package //lunabot_2425/stl/wheel_mo.stl"/> -->
         <cylinder radius="${whee_rad}" length="${whee_len}"/>
         <!-- <box size="${nuck_sx} ${nuck_sy} ${nuck_sz}"/> -->
@@ -439,5 +439,5 @@
     <visual>
       <geometry>
-        <!-- <mesh filename="package://lunabot_2425/stl/wheel_mo.stl"/> -->
+        <!-- <mesh filename="package //lunabot_2425/stl/wheel_mo.stl"/> -->
         <!-- <cylinder radius="${whee_rad}" length="${whee_len}"/> -->
         <box size="${nuck_sx} ${nuck_sy} ${nuck_sz}"/>
@@ -448,5 +448,5 @@
     <collision>
       <geometry>
-        <!-- <mesh filename="package://lunabot_2425/stl/wheel_mo.stl"/> -->
+        <!-- <mesh filename="package //lunabot_2425/stl/wheel_mo.stl"/> -->
         <cylinder radius="${whee_rad}" length="${whee_len}"/>
       </geometry>
